Commit message: feat: 实车导航稳定性优化与部署文档更新
- 重写 lidar_navigation_guide.md，补充 FAST-LIO/AMCL 多模式说明、一键启动与 RViz 操作
- 修复 betop_teleop README 中 /cmd_vel 话题名与格式错误，统一为 /cmd_vel_joy
- 修正 diuniu_teleop_cmd_vel.py 日志/注释中的话题名
- 新增 debug_weekly_report_v2.md 与 diuniu_nav_all.launch.py
- 删除过时的 task_handover.md
- 底盘驱动新增 20Hz 看门狗与 cmd_vel/cmd_vel_joy 双通道隔离
- 调整 URDF 雷达安装位置与 Nav2 参数适配实车

File: src/diuniu_description/urdf/diuniu.urdf (robot description, URDF)
Before this commit: robot diuniu, 6 links, 5 joints
Joints:
- joint laser_joint: origin xyz=1.25 0 0.6 rpy=0 0 0 -> xyz=1.215 0 0.6 rpy=0 0 0

Commit message: feat(导航): 优化 Nav2 避障急停、A* 混合规划、AMCL 抗人体干扰与车辆 1.90m 物理模型

File: src/diuniu_description/urdf/diuniu.urdf (robot description, URDF)
Before this commit: robot diuniu, 6 links, 5 joints
Links:
- link base_link: geometry visual box size=1.90 0.7 0.2
Joints:
- joint laser_joint: origin xyz=1.215 0 0.6 rpy=0 0 0 -> xyz=1.215 0 0.66 rpy=0 0 0

Commit message: feat(description): 更新雷达安装参数（高度 160cm，倒装 Roll=180度）

File: src/diuniu_description/urdf/diuniu.urdf (robot description, URDF)
Before this commit: robot diuniu, 6 links, 5 joints
Joints:
- joint laser_joint: origin xyz=1.215 0 0.66 rpy=0 0 0 -> xyz=1.215 0 1.60 rpy=3.14159265 0 0

Commit message: fix(description): 将 imu_link 的父坐标系修正绑定至 laser_link，使内置 IMU 正确继承 160cm 倒装 TF 变换

File: src/diuniu_description/urdf/diuniu.urdf (robot description, URDF)
Before this commit: robot diuniu, 6 links, 5 joints
Joints:
- joint imu_joint: origin xyz=0.675 0 0.2 rpy=0 0 0 -> xyz=0 0 0 rpy=0 0 0; parent base_link -> laser_link

Commit message: fix(nav&filter): 修正 pointcloud_to_laserscan 在 base_link 下的 min_height 为 0.20m，彻底消除车前地面弧形扫地虚假障碍物

File: src/diuniu_description/urdf/diuniu.urdf (robot description, URDF)
Before this commit: robot diuniu, 6 links, 5 joints
Links:
- added link base_imu_link; visual box size=0.05 0.05 0.02
Joints:
- added joint base_imu_joint: type fixed, parent base_link, child base_imu_link, origin xyz=0 0 0.10 rpy=0 0 0

Commit message: feat(n10): add N10 2D lidar navigation stack and tune parameters for DiNiu forklift

File: src/diuniu_description/urdf/diuniu.urdf (robot description, URDF)
Before this commit: robot diuniu, 7 links, 6 joints
Links:
- added link n10_laser_link; visual cylinder length=0.04 radius=0.028
Joints:
- added joint n10_laser_joint: type fixed, parent base_link, child n10_laser_link, origin xyz=1.295 0 0.66 rpy=0 0 0
- joint laser_joint: origin xyz=1.215 0 1.60 rpy=3.14159265 0 0 -> xyz=1.215 0 0.66 rpy=0 0 0
